File: hardware/electronics/SpotAI/SpotAI.kicad_pcb (KiCad board)
At the start: 2 copper layers, 70.1 x 79.9 mm, 9 parts, among them IC1 TEENSY3.2, J1 Respeaker, J2 motors, J3 mpu6050, J4 lid1, J5 lid2, J6 HC_SR04, J7 DHT22, J8 Jetson

Commit message: pcb_placement
Parts:
- J8: moved to B.Cu
- moved IC1 198.0 mm to (80.5, 121.0), turned to 0 degrees
- moved J4 189.6 mm to (79.8, 126.5), turned to 90 degrees
- moved J1 172.3 mm to (80.5, 100.1), turned to 180 degrees
- moved J8 159.6 mm to (93.2, 100.1), turned to 0 degrees
- moved J6 155.0 mm to (103.2, 126.7), turned to 270 degrees
- moved J5 151.5 mm to (128.8, 126.8), turned to 90 degrees
- moved J2 146.9 mm to (120.5, 126.8), turned to 270 degrees
- moved J7 133.3 mm to (122.2, 106.8)
- moved J3 132.1 mm to (121.9, 90.7)
Connections:
- J3 pad 3: SDA0 -> SCL0
- J3 pad 4: SCL0 -> SDA0
- J4 pad 3: SDA0 -> SCL0
- J4 pad 4: SCL0 -> SDA0
- J5 pad 3: SDA0 -> SCL0
- J5 pad 4: SCL0 -> SDA0
Other:
- board size 70.1 x 79.9 mm -> 77.6 x 86 mm

Commit message: pcb_root;gerber
Parts:
- added REF**: MountingHole_3.2mm_M3_Pad, MountingHole:MountingHole_3.2mm_M3_Pad, F.Cu at (146.3, 78.5)
- added REF**: MountingHole_3.2mm_M3_Pad, MountingHole:MountingHole_3.2mm_M3_Pad, F.Cu at (146.2, 110.5)
Connections:
- J2 pad 1: VCC -> +3V3
Routing:
- net (no net): track 0.00 -> 138.2 mm
- net +3V3: track 0.00 -> 111.6 mm
- net SCL0: track 0.00 -> 108.1 mm
- net SDA0: track 0.00 -> 104.4 mm
- net J_RX: track 0.00 -> 34.2 mm
- net DHT: track 0.00 -> 33.1 mm
- net VCC: track 0.00 -> 30.6 mm
- net J_TX: track 0.00 -> 30.6 mm
- net TRIG: track 0.00 -> 28.2 mm
- net Echo: track 0.00 -> 28.2 mm
- net GPIO12: track 0.00 -> 18.8 mm
- net I2S_DAC: track 0.00 -> 18.8 mm
- net CSO: track 0.00 -> 18.8 mm
- net I2S_CLK: track 0.00 -> 18.8 mm
- net I2S_ADC: track 0.00 -> 18.8 mm
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- added copper zone on B.Cu, net GND
- added copper zone on F.Cu, net GND
Other:
- outline, holes or cut-outs redrawn
- board text added: "Made by: benoitlx"
- board text added: "SpotAI"
