File: hardware/electronics/SpotAI/SpotAI.sch (KiCad schematic (older format))
At the start: 9 parts, among them IC1 TEENSY3.2, J1 Respeaker, J2 motors, J3 mpu6050, J4 lid1, J5 lid2, J6 HC_SR04, J7 DHT22, J8 Jetson

Commit message: pcb_placement
Connections:
- net SCL0: now also J3.3 (Pin_3), J4.3 (Pin_3), J5.3 (Pin_3); no longer J3.4 (Pin_4), J4.4 (Pin_4), J5.4 (Pin_4)
- net SDA0: now also J3.4 (Pin_4), J4.4 (Pin_4), J5.4 (Pin_4); no longer J3.3 (Pin_3), J4.3 (Pin_3), J5.3 (Pin_3)
Changed lines of the file:
@@
 SCL0
 Wire Wire Line
-	3400 3700 3600 3700
-Wire Wire Line
-	3400 3800 3650 3800
-Wire Wire Line
-	3600 3700 3600 4250
-Wire Wire Line
 	3600 4250 4000 4250
-Connection ~ 3600 3700
-Wire Wire Line
-	3600 3700 4000 3700
-Wire Wire Line
-	3650 3800 3650 4350
 Wire Wire Line
 	3650 4350 4000 4350
-Connection ~ 3650 3800
-Wire Wire Line
-	3650 3800 4000 3800
 Wire Wire Line
 	3600 4250 3600 4800
 Wire Wire Line
 	3600 4800 4000 4800
-Connection ~ 3600 4250
 Wire Wire Line
 	3650 4350 3650 4900
@@
 Wire Wire Line
 	9650 2350 9650 2200
+Connection ~ 3650 3700
+Wire Wire Line
+	3650 3700 4000 3700
+Wire Wire Line
+	3650 3700 3650 4350
+Wire Wire Line
+	3400 3800 3600 3800
+Wire Wire Line
+	3400 3700 3650 3700
+Wire Wire Line
+	3600 4250 3600 3800
+Connection ~ 3600 4250
+Connection ~ 3600 3800
+Wire Wire Line
+	3600 3800 4000 3800
 $EndSCHEMATC

Commit message: pcb_root;gerber
Parts:
- IC1: symbol TEENSY3.2:TEENSY3.2 -> SpotAI-rescue:TEENSY3.2-TEENSY3.2
Connections:
- net +3V3: now also J2.1 (Pin_1)
- net VCC: no longer J2.1 (Pin_1)
Changed lines of the file:
@@
 $EndDescr
 $Comp
-L TEENSY3.2:TEENSY3.2 IC1
+L SpotAI-rescue:TEENSY3.2-TEENSY3.2 IC1
 U 1 1 60FEE192
 P 5850 3550
@@
 $EndComp
 $Comp
-L power:VCC #PWR06
-U 1 1 610F23B3
-P 3700 3350
-F 0 "#PWR06" H 3700 3200 50  0001 C CNN
-F 1 "VCC" H 3800 3450 50  0000 C CNN
-F 2 "" H 3700 3350 50  0001 C CNN
-F 3 "" H 3700 3350 50  0001 C CNN
-	1    3700 3350
-	1    0    0    -1
-$EndComp
-Wire Wire Line
-	4000 3500 3700 3500
-Wire Wire Line
-	3700 3500 3700 3350
-$Comp
 L power:+3V3 #PWR05
 U 1 1 610F8F7A
@@
 $EndComp
 Wire Wire Line
-	3550 3350 3550 4050
+	3550 3350 3550 3500
 Wire Wire Line
 	3550 4600 4000 4600
@@
 Wire Wire Line
 	3600 3800 4000 3800
+Wire Wire Line
+	3550 3500 4000 3500
+Connection ~ 3550 3500
+Wire Wire Line
+	3550 3500 3550 4050
 $EndSCHEMATC
